File: Hardware/USB_Type_A_Female_Breakout.sch (EAGLE design)
At the start: 12 parts

Commit message: Moved USB jack back. Added 0 Ohm DNP resistor to optionally connect USB jack shield to GND.
Parts:
- added R1: 0, SparkFun-Resistors:RESISTOR0603
- JP1: value USB_ -> USB+SHIELDUSB-A-S-NOSILK-FEMALE; device SparkFun-Connectors:USB_ -> SparkFun-Connectors:USB+SHIELDUSB-A-S-NOSILK-FEMALE
Connections:
- new net N$1: JP1.S1, JP1.S2, R1.2
- net GND: now also R1.1
Changed lines of the file:
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@@
 <?xml version="1.0" encoding="utf-8"?>
 <!DOCTYPE eagle SYSTEM "eagle.dtd">
-<eagle version="6.0">
+<eagle version="6.5.0">
 <drawing>
 <settings>
@@
 <layers>
 <layer number="1" name="Top" color="4" fill="1" visible="no" active="no"/>
+<layer number="2" name="Route2" color="1" fill="3" visible="no" active="no"/>
+<layer number="3" name="Route3" color="4" fill="3" visible="no" active="no"/>
+<layer number="4" name="Route4" color="1" fill="4" visible="no" active="no"/>
+<layer number="5" name="Route5" color="4" fill="4" visible="no" active="no"/>
+<layer number="6" name="Route6" color="1" fill="8" visible="no" active="no"/>
+<layer number="7" name="Route7" color="4" fill="8" visible="no" active="no"/>
+<layer number="8" name="Route8" color="1" fill="2" visible="no" active="no"/>
+<layer number="9" name="Route9" color="4" fill="2" visible="no" active="no"/>
+<layer number="10" name="Route10" color="1" fill="7" visible="no" active="no"/>
+<layer number="11" name="Route11" color="4" fill="7" visible="no" active="no"/>
+<layer number="12" name="Route12" color="1" fill="5" visible="no" active="no"/>
+<layer number="13" name="Route13" color="4" fill="5" visible="no" active="no"/>
+<layer number="14" name="Route14" color="1" fill="6" visible="no" active="no"/>
+<layer number="15" name="Route15" color="4" fill="6" visible="no" active="no"/>
 <layer number="16" name="Bottom" color="1" fill="1" visible="no" active="no"/>
 <layer number="17" name="Pads" color="2" fill="1" visible="no" active="no"/>
@@
 <parts>
 <part name="FRAME1" library="SparkFun-Aesthetics" deviceset="FRAME-LETTER" device=""/>
-<part name="JP1" library="SparkFun-Connectors" deviceset="USB" device="_"/>
+<part name="JP1" library="SparkFun-Connectors" deviceset="USB+SHIELD" device="USB-A-S-NOSILK-FEMALE"/>
 <part name="JP2" library="SparkFun-Connectors" deviceset="M04" device="PTH"/>
 <part name="GND1" library="SparkFun-Aesthetics" deviceset="GND" device=""/>
@@
 <part name="LOGO2" library="SparkFun-Aesthetics" deviceset="OSHW-LOGO" device="S"/>
 <part name="LOGO3" library="SparkFun-Aesthetics" deviceset="LOGO-SFE" device="SK"/>
+<part name="R1" library="SparkFun-Resistors" deviceset="RESISTOR" device="0603" value="0">
+<attribute name="PLACE" value="DNP"/>
+</part>
+<part name="GND3" library="SparkFun-Aesthetics" deviceset="GND" device=""/>
 </parts>
 <sheets>
@@
 <instance part="LOGO2" gate="G$1" x="132.08" y="12.7"/>
 <instance part="LOGO3" gate="G$1" x="231.14" y="25.4"/>
+<instance part="R1" gate="G$1" x="106.68" y="83.82" smashed="yes" rot="R90">
+<attribute name="NAME" x="109.22" y="86.3346" size="1.778" layer="95"/>
+<attribute name="VALUE" x="109.22" y="81.28" size="1.778" layer="96"/>
+<attribute name="PLACE" x="109.22" y="83.82" size="1.778" layer="96"/>
+</instance>
+<instance part="GND3" gate="1" x="106.68" y="73.66"/>
 </instances>
 <busses>
@@
 <wire x1="134.62" y1="99.06" x2="134.62" y2="96.52" width="0.1524" layer="91"/>
 </segment>
-</net>
+<segment>
+<pinref part="R1" gate="G$1" pin="1"/>
+<wire x1="106.68" y1="78.74" x2="106.68" y2="76.2" width="0.1524" layer="91"/>
+<pinref part="GND3" gate="1" pin="GND"/>
+</segment>
+</net>
+<net name="N$1" class="0">
+<segment>
+<pinref part="JP1" gate="G$1" pin="S2"/>
+<wire x1="104.14" y1="93.98" x2="104.14" y2="91.44" width="0.1524" layer="91"/>
+<wire x1="104.14" y1="91.44" x2="106.68" y2="91.44" width="0.1524" layer="91"/>
+<pinref part="R1" gate="G$1" pin="2"/>
+<wire x1="106.68" y1="91.44" x2="106.68" y2="88.9" width="0.1524" layer="91"/>
+<pinref part="JP1" gate="G$1" pin="S1"/>
+<wire x1="106.68" y1="93.98" x2="106.68" y2="91.44" width="0.1524" layer="91"/>
+<junction x="106.68" y="91.44"/>
+</segment>
+</net>
